File: pcb/temper.kicad_pcb (KiCad board)
At the start: 2 copper layers, 111.3 x 90 mm, 48 parts, among them J2 nice_view, SW1 SW_PUSH, SW10 SW_PUSH, SW11 SW_PUSH, SW12 SW_PUSH, SW13 SW_PUSH, SW14 SW_PUSH, SW15 SW_PUSH, SW16 SW_PUSH, SW17 SW_PUSH, SW18 SW_PUSH, SW2 SW_PUSH, SW3 SW_PUSH, SW4 SW_PUSH, SW5 SW_PUSH, SW6 SW_PUSH, SW7 SW_PUSH, SW8 SW_PUSH, SW9 SW_PUSH, U1 nice_nano

Commit message: Add my version
Other:
- board text added: "temper @hrfmartins"
- board text removed: "temper @raeedcho"
